File: power-monitor/power-monitor.kicad_pcb (KiCad board)
At the start: 2 copper layers, 40 x 17 mm, 16 parts, among them J1 Conn_01x02, J2 Conn_01x02, J3 Conn_01x05, Q1 IRF7403, U1 INA220

Commit message: Fix soldermask clearance
Other:
- rule pad_to_mask_clearance: 0.051 -> 0
